Commit message: Added tenacity_watchdog_manager: Tilt-sensor & cliff sensor code. The tilt sensor is the most complete and generally usable as-is. The others are a bit of a mix of Tenacity-specific and works-in-progress

File: tenacity_description/urdf/astra.xacro (robot description, xacro)
@@ -29,4 +29,30 @@
       <gazebo reference="astra">
           <material>Gazebo/White</material>
+          <plugin name="camera_plugin" filename="libgazebo_ros_openni_kinect.so">
+           <baseline>0.2</baseline>
+           <alwaysOn>true</alwaysOn>
+           <!-- Keep this zero, update_rate in the parent <sensor> tag
+             will control the frame rate. -->
+           <updateRate>0.0</updateRate>
+           <cameraName>camera_ir</cameraName>
+           <imageTopicName>/camera/color/image_raw</imageTopicName>
+           <cameraInfoTopicName>/camera/color/camera_info</cameraInfoTopicName>
+           <depthImageTopicName>/camera/depth/image_raw</depthImageTopicName>
+           <depthImageCameraInfoTopicName>/camera/depth/camera_info</depthImageCameraInfoTopicName>
+           <pointCloudTopicName>/camera/depth/points</pointCloudTopicName>
+           <frameName>camera_link</frameName>
+           <pointCloudCutoff>0.5</pointCloudCutoff>
+           <pointCloudCutoffMax>3.0</pointCloudCutoffMax>
+           <distortionK1>0</distortionK1>
+           <distortionK2>0</distortionK2>
+           <distortionK3>0</distortionK3>
+           <distortionT1>0</distortionT1>
+           <distortionT2>0</distortionT2>
+           <CxPrime>0</CxPrime>
+           <Cx>0</Cx>
+           <Cy>0</Cy>
+           <focalLength>0</focalLength>
+           <hackBaseline>0</hackBaseline>
+         </plugin>
       </gazebo>
       <gazebo reference="astra_joint">

File: tenacity_description/urdf/tenacity.urdf.xacro (robot description, xacro)
@@ -40,4 +40,5 @@
     <xacro:include filename="$(find tenacity_description)/urdf/mast_mount.xacro"/>
     <xacro:include filename="$(find tenacity_description)/urdf/astra.xacro"/>
+    <!-- <xacro:include filename="$(find tenacity_description)/urdf/tenacity_astra.xacro"/> -->
     <!-- Gazebo plugins -->
     <gazebo>

File: tenacity_description/urdf/tenacity_astra.xacro (robot description, xacro)
@@ -11,5 +11,5 @@
                 <origin rpy="0 0 0" xyz="0 0 0" />
                 <geometry>
-                    <mesh filename="package://tenacity_description/meshes/sensors/astra-camera.stl" />
+                   <mesh filename="package://tenacity_description/meshes/sensors/astra-camera.stl" />
                 </geometry>
                 <material name="grey" />
@@ -36,5 +36,5 @@
                </clip>
              </camera>
-             <plugin name="astra_camera_controller" filename="libgazebo_ros_openni_kinect.so">
+         <plugin name="camera_plugin" filename="libgazebo_ros_openni_kinect.so">
           <baseline>0.2</baseline>
           <alwaysOn>true</alwaysOn>
@@ -65,7 +65,7 @@
         </gazebo>
     </xacro:macro>
-    <xacro:macro name="astra_joint" params="x y z p" >
+    <xacro:macro name="astra_joint" params="x y z roll pitch yaw" >
         <joint name="astra_joint" type="fixed">
-		<origin rpy="0 ${p} 0" xyz="${x} ${y} ${z}"/>
+		<origin rpy="${roll} ${pitch} ${yaw}" xyz="${x} ${y} ${z}"/>
             <parent link="base_link" />
             <child link="astra" />

Commit message: Bulk update, including support for OAK-D stereocam in Gazebo

File: tenacity_description/urdf/astra.xacro (robot description, xacro)
@@ -6,11 +6,12 @@
       <xacro:property name="astra_depth" value="0.050" />
       <xacro:property name="astra_mass" value="0.15" />
+    <xacro:include filename="$(find tenacity_description)/urdf/astra.gazebo" />
     <xacro:macro name="astra_link">
       <link name="astra">
+              <pose>0.0 0.0 0.0 0.0 0.0 0.0</pose>
           <visual>
-              <origin rpy="0 0 0" xyz="0 0 0" />
+              <origin rpy="0 0 0" xyz="-0.05 0 0" />
               <geometry>
-                  <mesh filename="package://tenacity_description/meshes/sensors/astra-cam.stl" scale="0.001 0.001 0.001"/>
-                  <!-- <box size="${astra_length} ${astra_width} ${astra_depth}"/> -->
+                     <mesh filename="package://tenacity_description/meshes/sensors/orbbec_astra_camera.dae"/>
               </geometry>
               <material name="green" />
@@ -27,33 +28,13 @@
               x="${astra_length}" y="${astra_width}" z="${astra_depth}" />
       </link>
-      <gazebo reference="astra">
-          <material>Gazebo/White</material>
-          <plugin name="camera_plugin" filename="libgazebo_ros_openni_kinect.so">
-           <baseline>0.2</baseline>
-           <alwaysOn>true</alwaysOn>
-           <!-- Keep this zero, update_rate in the parent <sensor> tag
-             will control the frame rate. -->
-           <updateRate>0.0</updateRate>
-           <cameraName>camera_ir</cameraName>
-           <imageTopicName>/camera/color/image_raw</imageTopicName>
-           <cameraInfoTopicName>/camera/color/camera_info</cameraInfoTopicName>
-           <depthImageTopicName>/camera/depth/image_raw</depthImageTopicName>
-           <depthImageCameraInfoTopicName>/camera/depth/camera_info</depthImageCameraInfoTopicName>
-           <pointCloudTopicName>/camera/depth/points</pointCloudTopicName>
-           <frameName>camera_link</frameName>
-           <pointCloudCutoff>0.5</pointCloudCutoff>
-           <pointCloudCutoffMax>3.0</pointCloudCutoffMax>
-           <distortionK1>0</distortionK1>
-           <distortionK2>0</distortionK2>
-           <distortionK3>0</distortionK3>
-           <distortionT1>0</distortionT1>
-           <distortionT2>0</distortionT2>
-           <CxPrime>0</CxPrime>
-           <Cx>0</Cx>
-           <Cy>0</Cy>
-           <focalLength>0</focalLength>
-           <hackBaseline>0</hackBaseline>
-         </plugin>
-      </gazebo>
+<!--
+      <joint name="camera_optical_joint" type="fixed">
+         <origin xyz="0.00 0 0.00" rpy="${-pi/2} 0 ${-pi/2}"/>
+         <parent link="astra"/>
+         <child link="camera_link_optical"/>
+      </joint>
+  <link name="camera_link_optical">
+  </link>
+-->
       <gazebo reference="astra_joint">
           <!-- <disableFixedJointLumping>true</disableFixedJointLumping>  -->

File: tenacity_description/urdf/tenacity.urdf.xacro (robot description, xacro)
@@ -37,8 +37,14 @@
     <xacro:include filename="$(find tenacity_description)/urdf/tenacity_laser.xacro"/>
     <xacro:include filename="$(find tenacity_description)/urdf/tenacity_imu.xacro"/>
-    <xacro:include filename="$(find tenacity_description)/urdf/sensor_stalk.xacro"/>
+    <!--    <xacro:include filename="$(find tenacity_description)/urdf/sensor_stalk.xacro"/> -->
     <xacro:include filename="$(find tenacity_description)/urdf/mast_mount.xacro"/>
-    <xacro:include filename="$(find tenacity_description)/urdf/astra.xacro"/>
-    <!-- <xacro:include filename="$(find tenacity_description)/urdf/tenacity_astra.xacro"/> -->
+    <!--    <xacro:include filename="$(find tenacity_description)/urdf/astra.xacro"/> -->
+    <!-- <xacro:include filename="$(find tenacity_description)/urdf/oakd.xacro"/> -->
+    <!-- <xacro:include filename="$(find tenacity_description)/urdf/tenacity_oakd.xacro"/> -->
+    <xacro:include filename="$(find tenacity_description)/urdf/tenacity_oakd_multicamera.xacro"/>
+    <xacro:include filename="$(find tenacity_description)/urdf/oakd_mount.xacro"/>
+    <xacro:include filename="$(find tenacity_description)/urdf/front_cover.xacro"/>
+    <xacro:include filename="$(find tenacity_description)/urdf/tenacity_sonar.xacro"/>
+    <xacro:include filename="$(find tenacity_description)/urdf/tenacity_hazcam.xacro"/>
     <!-- Gazebo plugins -->
     <gazebo>
@@ -86,5 +92,5 @@
     <xacro:property name="body_box_width" value="0.285" />
     <xacro:property name="body_box_depth" value="0.093" />
-    <xacro:property name="body_box_mass" value="1.0" />
+    <xacro:property name="body_box_mass" value="1.00" />
     <xacro:property name="front_rocker_arm_length" value="0.182" />
     <xacro:property name="back_rocker_arm_length" value="0.161" />
@@ -342,4 +348,28 @@
             <material>Gazebo/Green</material>
         </gazebo>
+      </xacro:macro>
+    <xacro:macro name="corner_link_box" params="lon_label lat_label reflect">
+        <link name="${lon_label}_${lat_label}_corner_link_box">
+            <visual>
+                <origin rpy="0 0 0" xyz="0.05 0 0.05" />
+                <geometry>
+                     <box size="0.1 0.1 0.1"/>
+                </geometry>
+                <material name="blue" />
+            </visual>
+            <collision>
+                <origin rpy="0 0 0" xyz="0 0 0" />
+                <geometry>
+                    <box size="0.1 0.1 0.1"/>
+                </geometry>
+            </collision>
+            <xacro:solid_cuboid_inertial
+                rpy="0 0 0" xyz="0 0 0"
+                mass="0.25"
+                x="0.1" y="0.1" z="0.1" />
+        </link>
+        <gazebo reference="${lon_label}_${lat_label}_corner_link_box">
+            <material>Gazebo/Blue</material>
+        </gazebo>
     </xacro:macro>
     <xacro:corner_link lon_label="front" lat_label="left" reflect="1"/>
@@ -529,13 +559,34 @@
     <xacro:corner_wheel_joint lon_label="back" lat_label="left" reflect="1"/>
     <xacro:corner_wheel_joint lon_label="back" lat_label="right" reflect="-1"/>
-    <!-- Laser Scan Sensor -->
-    <xacro:astra_link />
-    <xacro:astra_joint x="0.240" y="0.005" z="0.154" roll="0.17" pitch="0.00" yaw="1.57" />
+    <!-- AstraCam -->
+    <!--    <xacro:astra_link />  -->
+    <!-- <xacro:astra_joint x="0.3080" y="0.005" z="0.170" roll="0.00" pitch="0.00" yaw="0.00" /> -->
     <!-- Antenna/Sensor Mast -->
     <xacro:mast_mount_link />
     <xacro:mast_mount_joint x="-0.152" y="-0.090" z="0.050" />
      <!-- SensorStalk -->
-     <xacro:sensor_stalk_link />
-     <xacro:sensor_stalk_joint x="0.2280" y="0.005" z="0.0320" />
+     <xacro:oakd_mount_link />
+     <xacro:oakd_mount_joint x="0.2380" y="-0.004" z="0.0320" />
+     <xacro:oakd_link mount_point="main" />
+     <!-- <xacro:oakd_joint x="0.2850" y="-0.006" z="0.2080"  roll="1.5757" pitch="0.00" yaw="1.5757" mount_point="main"/> -->
+     <xacro:oakd_joint x="0.2850" y="-0.006" z="0.2080"  roll="0.00" pitch="0.00" yaw="0.00" mount_point="main"/>
+     <xacro:front_cover_link />
+     <xacro:front_cover_joint x="0.150" y="0.00" z="-0.0180"  roll="0" pitch="0.00" yaw="0"/>
+     <!-- Sonar Sensor -->
+     <xacro:sonar_link mount_point="cliff"/>
+     <xacro:sonar_joint x="0.230" y="0.005" z="-0.0320" roll="0.00" pitch="0.4" yaw="0.00" mount_point="cliff"/>
+     <xacro:sonar_link mount_point="forward"/>
+     <xacro:sonar_joint x="0.250" y="0.00" z="0.0420" roll="0.00" pitch="0.0" yaw="0.00" mount_point="forward"/>
+     <xacro:sonar_link mount_point="left"/>
+     <xacro:sonar_joint x="0.285" y="0.2559" z="0.0180" roll="0.00" pitch="0" yaw="0.65" mount_point="left"/>
+     <xacro:sonar_link mount_point="right"/>
+     <xacro:sonar_joint x="0.285" y="-0.2559" z="0.0180" roll="0.00" pitch="0" yaw="-0.65" mount_point="right"/>
+     <!-- Hazard Cameras -->
+     <!--     <xacro:hazcam_link mount_point="left"/> -->
+     <!-- <xacro:hazcam_joint x="0.295" y="0.2559" z="0.0180" roll="0.00" pitch="0" yaw="1.5757" mount_point="left"/> -->
+     <!--  <xacro:hazcam_link mount_point="right"/> -->
+     <!--   <xacro:hazcam_joint x="0.295" y="-0.2559" z="0.0180" roll="0.00" pitch="0" yaw="-1.5757" mount_point="right"/> -->
+     <!--   <xacro:hazcam_link mount_point="forward"/> -->
+     <!--   <xacro:hazcam_joint x="0.31" y="0.003" z="0.0080" roll="0.00" pitch="0" yaw="0" mount_point="forward"/> -->
      <!-- IMU -->
      <xacro:imu_link />

File: tenacity_description/urdf/tenacity_astra.xacro (robot description, xacro)
@@ -36,30 +36,4 @@
                </clip>
              </camera>
-         <plugin name="camera_plugin" filename="libgazebo_ros_openni_kinect.so">
-          <baseline>0.2</baseline>
-          <alwaysOn>true</alwaysOn>
-          <!-- Keep this zero, update_rate in the parent <sensor> tag
-            will control the frame rate. -->
-          <updateRate>0.0</updateRate>
-          <cameraName>camera_ir</cameraName>
-          <imageTopicName>/camera/color/image_raw</imageTopicName>
-          <cameraInfoTopicName>/camera/color/camera_info</cameraInfoTopicName>
-          <depthImageTopicName>/camera/depth/image_raw</depthImageTopicName>
-          <depthImageCameraInfoTopicName>/camera/depth/camera_info</depthImageCameraInfoTopicName>
-          <pointCloudTopicName>/camera/depth/points</pointCloudTopicName>
-          <frameName>camera_link</frameName>
-          <pointCloudCutoff>0.5</pointCloudCutoff>
-          <pointCloudCutoffMax>3.0</pointCloudCutoffMax>
-          <distortionK1>0</distortionK1>
-          <distortionK2>0</distortionK2>
-          <distortionK3>0</distortionK3>
-          <distortionT1>0</distortionT1>
-          <distortionT2>0</distortionT2>
-          <CxPrime>0</CxPrime>
-          <Cx>0</Cx>
-          <Cy>0</Cy>
-          <focalLength>0</focalLength>
-          <hackBaseline>0</hackBaseline>
-        </plugin>
          </sensor>
         </gazebo>
