Commit message: updated OAKD xacro to include dummy links/joints for processing pointclouds generated from stereo_image_proc

File: tenacity_description/urdf/tenacity_oakd_multicamera.xacro (robot description, xacro)
@@ -27,4 +27,18 @@
               x="${oakd_length}" y="${oakd_width}" z="${oakd_depth}" />
       </link>
+      <!-- Add dummy joint for camera_optical_frame to link back to base_link -->
+        <joint name="camera_optical_joint" type="fixed">
+           <origin rpy="-1.57079632769 0 -1.570796332769" xyz="0 0 0" />
+	   <parent link="oakd_${mount_point}" />
+	   <child link="camera_optical_frame" />
+	</joint>
+	<!-- Add dummy link for camera_optical_frame to link back to base_link -->
+        <link name="camera_optical_frame">
+        <inertial>
+	  <mass value="0.001" />
+	  <origin xyz="0 0 0" />
+	  <inertia ixx="0.0001" ixy="0.0" ixz="0.0" iyy="0.0001" iyz="0.0" izz="0.0001" />
+          </inertial>
+          </link>
       <gazebo reference="oakd_${mount_point}">
     <material>Gazebo/DarkGrey</material>
@@ -40,6 +54,6 @@
         </image>
         <clip>
-          <near>0.02</near>
-          <far>300</far>
+          <near>0.3</near>
+          <far>35</far>
         </clip>
         <noise>
@@ -59,6 +73,6 @@
         </image>
         <clip>
-          <near>0.02</near>
-          <far>300</far>
+          <near>0.3</near>
+          <far>35</far>
         </clip>
         <noise>
