Commit message: Fixed syntax error in the OAKD XACRO file(s) that was causing the OAKD camera model to not appear in Gazebo

File: tenacity_description/urdf/oakd_multicamera.xacro (robot description, xacro)
@@ -90,5 +90,5 @@
     <xacro:macro name="oakd_joint" params="x y z roll pitch yaw mount_point" >
         <joint name="oakd_joint_${mount_point}" type="fixed">
-                <origin rpy="${roll} ${pitch} ${yaw}" xyz="${x}+0.1 ${y}-0.01 ${z}"/>
+                <origin rpy="${roll} ${pitch} ${yaw}" xyz="${x+0.1} ${y-0.01} ${z}"/>
             <parent link="base_link" />
             <child link="oakd_${mount_point}" />

File: tenacity_description/urdf/tenacity.urdf.xacro (robot description, xacro)
@@ -37,5 +37,5 @@
     <xacro:include filename="$(find tenacity_description)/urdf/tenacity_laser.xacro"/>
     <xacro:include filename="$(find tenacity_description)/urdf/tenacity_imu.xacro"/>
-    <!--    <xacro:include filename="$(find tenacity_description)/urdf/sensor_stalk.xacro"/> -->
+    <xacro:include filename="$(find tenacity_description)/urdf/sensor_stalk.xacro"/>
     <xacro:include filename="$(find tenacity_description)/urdf/mast_mount.xacro"/>
     <!--    <xacro:include filename="$(find tenacity_description)/urdf/astra.xacro"/> -->
@@ -567,6 +567,5 @@
      <!-- SensorStalk -->
      <xacro:oakd_link mount_point="main" />
-     <!-- <xacro:oakd_joint x="0.2850" y="-0.006" z="0.2080"  roll="1.5757" pitch="0.00" yaw="1.5757" mount_point="main"/> -->
-     <xacro:oakd_joint x="0.2850" y="-0.006" z="0.2080"  roll="0.00" pitch="0.00" yaw="0.00" mount_point="main"/>
+     <xacro:oakd_joint x="0.270" y="0.002" z="0.1850"  roll="0.00" pitch="0.00" yaw="0.00" mount_point="main"/>
      <xacro:front_cover_link />
      <xacro:front_cover_joint x="0.150" y="0.00" z="-0.0180"  roll="0" pitch="0.00" yaw="0"/>

File: tenacity_description/urdf/tenacity_oakd_multicamera.xacro (robot description, xacro)
@@ -106,5 +106,5 @@
     <xacro:macro name="oakd_joint" params="x y z roll pitch yaw mount_point" >
         <joint name="oakd_joint_${mount_point}" type="fixed">
-                <origin rpy="${roll} ${pitch} ${yaw}" xyz="${x}+0.1 ${y}-0.01 ${z}"/>
+                <origin rpy="${roll} ${pitch} ${yaw}" xyz="${x} ${y} ${z}"/>
             <parent link="base_link" />
             <child link="oakd_${mount_point}" />
